File: BenchBudEE/$FanDriver.sch (KiCad schematic (older format))
At the start: 10 parts, among them Q2 MOSFET_N, Q3 MOSFET_N, Q4 MOSFET_N, U3 MCP4922-E/P, U4 OPA4170

Commit message: Parts added to thermocouple module. Relay & thermocouple rough placement.
Parts:
- U4: Distributor (none) -> DigiKey; Distributor Part Link (none) -> www.digikey.com/product-detail/en/OPA4170AIDR/296-29664-1-N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; Distributor Part Number (none) -> 296-29664-1-ND; MFG Name (none) -> Texas Instruments; MFG Part Number (none) -> OPA4170AIDR
Changed lines of the file:
@@
 F 1 "OPA4170" H 6300 1850 50  0000 C CNN
 F 2 "" H 6150 2050 60  0000 C CNN
-F 3 "" H 6150 2050 60  0000 C CNN
+F 3 "http://www.ti.com/lit/ds/symlink/opa4170.pdf" H 6150 2050 60  0001 C CNN
+F 4 "Texas Instruments" H 6150 2050 60  0001 C CNN "MFG Name"
+F 5 "OPA4170AIDR" H 6150 2050 60  0001 C CNN "MFG Part Number"
+F 6 "DigiKey" H 6150 2050 60  0001 C CNN "Distributor"
+F 7 "296-29664-1-ND" H 6150 2050 60  0001 C CNN "Distributor Part Number"
+F 8 "www.digikey.com/product-detail/en/OPA4170AIDR/296-29664-1-ND/2762167" H 6150 2050 60  0001 C CNN "Distributor Part Link"
 	3    6150 2050
 	1    0    0    -1
